File: Latch-Circuit/Latch-Circuit.kicad_sch (KiCad schematic)
At the start: 67 parts, among them J1 2-1445052-2, J2 3-794633-8, J3 B2P-VH, J4 3-794633-6, Q1 DMP3098LQ-7, Q2 2N7002K-AU_R1_000A2, Q3 2N7002K-AU_R1_000A2, Q4 2N7002K-AU_R1_000A2, U1 TLP3106A(TP,F, U2 TLP3106A(TP,F, U3 TLP3106A(TP,F, U4 CD4043BPWR, U5 TBD62003AFNG,EL

Commit message: ランプチェック回路を追加
Parts:
- added C1, C4: 0.1u, ProjectEV_Capacitor:C_1608M, symbol ProjectEV_Capacitor:C_1608M
- added C2: 10u, ProjectEV_Capacitor:C_1608M, symbol ProjectEV_Capacitor:C_1608M
- added C3: 1u, ProjectEV_Capacitor:C_2012M, symbol ProjectEV_Capacitor:C_2012M
- added C6: 10n, ProjectEV_Capacitor:C_1608M, symbol ProjectEV_Capacitor:C_1608M
- added D2: 1N4448WQ-7-F, ProjectEV_Diode:1N4448WQ-7-F, symbol ProjectEV_Diode:1N4448WQ-7-F
- added R1, R6: 100k, ProjectEV_Resistor:R_1608M, symbol ProjectEV_Resistor:R_1608M
- added R2: 360k, ProjectEV_Resistor:R_1608M, symbol ProjectEV_Resistor:R_1608M
- added U1: TLC555QDRQ1, ProjectEV_Timer:TLC555QDRQ1, symbol ProjectEV_Timer:TLC555QDRQ1
- renumbered C6 to C10, C3 to C11, C7 to C12, C2 to C5, C1 to C7, C4 to C8, C5 to C9, D3 to D1, D9 to D10, D1 to D3, D2 to D4, D4 to D5, D5 to D6, D6 to D7, D7 to D8, D8 to D9, J4 to J3, J3 to J4, R13 to R10, R16 to R11, R31 to R12, R11 to R13, R32 to R14, R14 to R15, R33 to R16, R9 to R18, R12 to R19, R15 to R20, R27 to R21, R19 to R22, R22 to R23, R25 to R24, R20 to R25, R23 to R26, R26 to R27, R18 to R28, R21 to R29, R6 to R3, R24 to R30, R3 to R31, R4 to R32, R28 to R33, R5 to R34, R29 to R35, R30 to R36, R7 to R4, R1 to R5, R8 to R7, R2 to R8, R10 to R9, U4 to U2, U5 to U3, U1 to U4, U2 to U5, U3 to U6
Connections:
- net +12V: now also C3.2, C4.1, R1.2, R2.2, R6.1, U1.4 (~{RESET}), U1.8 (VDD)
- net GND: now also C1.1, C2.1, C3.1, C4.2, C6.1, U1.1 (GND)
- net RST_SW2: now also D2.1 (K)
- new net: C2.2, R2.1, U1.6 (THRES), U1.7 (DISCH)
- new net: C1.2, R1.1, U1.2 (TRIG)
- new net: C6.2, U1.5 (CONT)
- new net LampCheck_SIG: D2.2 (A), R6.2, U1.3 (OUT)
Other:
- note added: "ランプチェック回路"
- note added: "点灯時間t = 1.1 × R56 × C31 = 1.1 × 360k × 10u ≈ 3.96 s"
- moved on the sheet: C10, C11, C12, C8, C9, D10, D5, D6, D7, D8, D9, H1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
Changed lines of the file:
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@@
 (kicad_sch
-	(version 20250114)
+	(version 20260306)
 	(generator "eeschema")
-	(generator_version "9.0")
-	(paper "A4")
+	(generator_version "10.0")
+	(paper "A3")
 	(title_block
 		(title "Latch-Circuit")
